File: pcb/magic_counter.kicad_pcb (KiCad board)
At the start: 2 copper layers, 127.4 x 202.4 mm, 182 parts, among them J1 ISP-Port, Q1 2SA1015, Q10 2SA1015, Q11 2SA1015, Q12 2SA1015, Q13 2SA1015, Q14 2SA1015, Q15 2SA1015, Q16 2SA1015, Q17 2SA1015, Q18 2SA1015, Q19 2SA1015, Q2 2SA1015, Q20 2SA1015, Q3 2SA1015, Q4 2SA1015, Q5 2SA1015, Q6 2SA1015, Q7 2SA1015, Q8 2SA1015, Q9 2SA1015, SW1 Reset, SW10 +1, SW11 +10, SW12 -10, SW13 -1, SW14 x2, SW15 /2, SW16 Random, SW2 +1, SW3 +10, SW4 -10, SW5 -1, SW6 x2, SW7 /2, SW8 Random, SW9 Reset, U1 ATmega32A-P, U10 74HC595, U11 4028, U12 LTC-4627JF, U13 LTC-4627JF, U2 74HC595, U3 74HC595, U4 4028, U5 LTC-4627JF, U6 LTC-4627JF, U7 74HC165, U8 74HC165, U9 74HC595, Y1 Crystal

Commit message: new tighter layout
Parts:
- moved SW25 183.7 mm to (37.6, 192.7)
- moved SW29 172.6 mm to (37.6, 205.1)
- moved SW30 161.0 mm to (50.7, 205.0)
- moved SW27 158.8 mm to (64.1, 193.2)
- moved Q16 147.6 mm to (91.4, 181.6)
- moved SW26 145.4 mm to (50.7, 192.9)
- moved Q17 142.4 mm to (102.1, 181.6)
- moved R76 141.9 mm to (99.2, 199.8), turned to 180 degrees
- moved U15 140.8 mm to (123.3, 195.4)
- moved R52 140.2 mm to (47.5, 200.2), turned to 90 degrees
- moved C17 138.8 mm to (119.5, 190.5), turned to 90 degrees
- moved R53 137.3 mm to (60.8, 200.1), turned to 90 degrees
- moved R80 133.0 mm to (111.9, 200.2), turned to 180 degrees
- moved C18 132.4 mm to (119.5, 192.8), turned to -90 degrees
- moved R56 128.8 mm to (47.5, 212.0), turned to 90 degrees
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Connections:
- R68 pad 2: Net-(Q15-Pad3) -> Net-(Q11-Pad3)
- R69 pad 2: Net-(Q14-Pad3) -> Net-(Q12-Pad3)
- R71 pad 2: Net-(Q12-Pad3) -> Net-(Q14-Pad3)
- R72 pad 2: Net-(Q11-Pad3) -> Net-(Q15-Pad3)
- R81 pad 2: Net-(Q20-Pad3) -> Net-(Q16-Pad3)
- R82 pad 2: Net-(Q19-Pad3) -> Net-(Q17-Pad3)
- R84 pad 2: Net-(Q17-Pad3) -> Net-(Q19-Pad3)
- R85 pad 2: Net-(Q16-Pad3) -> Net-(Q20-Pad3)
- U12 pad 1: Net-(Q15-Pad2) -> Net-(Q11-Pad2)
- U12 pad 2: Net-(Q14-Pad2) -> Net-(Q12-Pad2)
- U12 pad 4: Net-(Q11-Pad2) -> Net-(Q15-Pad2)
- U12 pad 8: Net-(Q12-Pad2) -> Net-(Q14-Pad2)
- U13 pad 1: Net-(Q20-Pad2) -> Net-(Q16-Pad2)
- U13 pad 2: Net-(Q19-Pad2) -> Net-(Q17-Pad2)
- U13 pad 4: Net-(Q16-Pad2) -> Net-(Q20-Pad2)
- U13 pad 8: Net-(Q17-Pad2) -> Net-(Q19-Pad2)
Routing:
- added copper zone on B.Cu, net GND

Commit message: fewer parts and reduced to prototyping board with more logic analyzer pins
Parts:
- removed C15, C16, C17, C18: ~, Capacitor_THT:C_Disc_D3.8mm_W2.6mm_P2.50mm
- removed C19, C21, C23: 100pF, Capacitor_THT:C_Disc_D3.8mm_W2.6mm_P2.50mm
- removed C20, C22, C24: 1nF, Capacitor_THT:C_Disc_D3.8mm_W2.6mm_P2.50mm
- removed Q10, Q11, Q12, Q13, Q14, Q15, Q16, Q17, Q18, Q19, Q20, Q9: 2SA1015, Package_TO_SOT_THT:TO-92_Wide
- removed R44, R45, R46, R47, R48, R49, R50, R51, R52, R53, R54, R55, R56, R57, R58, R59: 10k, Resistor_THT:R_Axial_DIN0207_L6.3mm_D2.5mm_P7.62mm_Horizontal
- removed R60, R61, R62, R63, R64, R65, R66, R67, R73, R74, R75, R76, R77, R78, R79, R80: 100R, Resistor_THT:R_Axial_DIN0207_L6.3mm_D2.5mm_P7.62mm_Horizontal
- removed R68, R69, R70, R71, R72, R81, R82, R83, R84, R85: 4.7k, Resistor_THT:R_Axial_DIN0207_L6.3mm_D2.5mm_P7.62mm_Horizontal
- removed SW18, SW19, SW20, SW21, SW22, SW23, SW24, SW25, SW26, SW27, SW28, SW29, SW30, SW31, SW32: ~, Button_Switch_THT:SW_PUSH_6mm_H5mm
- removed U10, U9: 74HC595, Package_DIP:DIP-16_W7.62mm_LongPads
- removed U11: 4028, Package_DIP:DIP-16_W7.62mm_LongPads
- removed U12, U13: LTC-4627JF, Display_7Segment:LTC-4627Jx
- removed U14, U15: ~, Package_DIP:DIP-16_W7.62mm_LongPads
- added J2: Serial Out, Connector_PinHeader_2.54mm:PinHeader_1x04_P2.54mm_Vertical, F.Cu at (66.2, 160.1)
- added J3: 1st Bit_shifter, Connector_PinHeader_2.54mm:PinHeader_1x03_P2.54mm_Vertical, F.Cu at (47.7, 85.4)
- added J4: 1st 7 Segment, Connector_PinHeader_2.54mm:PinHeader_1x08_P2.54mm_Vertical, F.Cu at (86.3, 97.9)
- C1: value 100pF -> 1nF
- C2: value 1nF -> 100pF
- Q1, Q2, Q3, Q4, Q5, Q6, Q7, Q8: value 2SA1015 -> Q_NPN_CBE; footprint Package_TO_SOT_THT:TO-92_Wide -> Package_TO_SOT_THT:TO-92_Inline_Wide
- R10, R11, R12, R13, R14: value 4.7k -> 100R
- R15, R16, R17, R18, R19: value 10k -> 100R
- R2, R3: value 100R -> 1k
- R20, R21, R22: value 10k -> 4.7k
- R23, R24, R25, R26, R27: value 100R -> 4.7k
- R28, R29, R30: value 100R -> 10k
- R31, R32, R33, R34, R35: value 4.7k -> 10k
- SW1, SW9: value Reset -> Random
- SW10, SW2: value +1 -> Reset
- SW11, SW3: value +10 -> +1
- SW12, SW4: value -10 -> +10
- SW13, SW5: value -1 -> -10
- SW14, SW6: value x2 -> -1
- SW15, SW7: value /2 -> x2
- SW16, SW8: value Random -> /2
- SW17: value ~ -> Random
- U5, U6: value LTC-4627JF -> CC56-12SURKWA; footprint Display_7Segment:LTC-4627Jx -> Display_7Segment:CA56-12SURKWA
- moved R35 265.5 mm to (290.0, 178.8), turned to 0 degrees
- moved SW17 264.8 mm to (301.2, 174.7)
- moved R34 258.3 mm to (290.0, 174.7), turned to 0 degrees
- moved R17 177.2 mm to (304.5, 108.1)
- moved R38 177.2 mm to (304.5, 147.7)
- moved R42 177.2 mm to (304.5, 159.3)
- moved C1 177.2 mm to (255.4, 151.7)
- moved C10 177.2 mm to (263.5, 117.2)
- moved C11 177.2 mm to (270.1, 130.4)
- moved C12 177.2 mm to (270.1, 127.8)
- moved C2 177.2 mm to (250.3, 151.7)
- moved C5 177.2 mm to (263.5, 105.6)
- moved C6 177.2 mm to (263.5, 103.0)
- moved C9 177.2 mm to (263.5, 114.6)
- moved Q5 177.2 mm to (218.1, 103.5)
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Connections:
- Q1 pad 1: +5V -> Net-(U5-Pad6)
- Q1 pad 2: Net-(Q1-Pad2) -> Net-(R20-Pad2)
- Q1 pad 3: Net-(Q1-Pad3) -> GND
- Q2 pad 1: +5V -> Net-(U5-Pad8)
- Q2 pad 2: Net-(Q2-Pad2) -> Net-(R21-Pad2)
- Q2 pad 3: Net-(Q2-Pad3) -> GND
- Q3 pad 1: +5V -> Net-(U5-Pad9)
- Q3 pad 2: Net-(Q3-Pad2) -> Net-(R22-Pad2)
- Q3 pad 3: Net-(Q3-Pad3) -> GND
- Q4 pad 1: +5V -> Net-(U5-Pad12)
- Q4 pad 2: Net-(Q4-Pad2) -> Net-(R23-Pad2)
- Q4 pad 3: Net-(Q4-Pad3) -> GND
- Q5 pad 1: +5V -> Net-(U6-Pad6)
- Q5 pad 2: Net-(Q5-Pad2) -> Net-(R24-Pad2)
- Q5 pad 3: Net-(Q5-Pad3) -> GND
- Q6 pad 1: +5V -> Net-(U6-Pad8)
- Q6 pad 2: Net-(Q6-Pad2) -> Net-(R25-Pad2)
- Q6 pad 3: Net-(Q6-Pad3) -> GND
- Q7 pad 1: +5V -> Net-(U6-Pad9)
- Q7 pad 2: Net-(Q7-Pad2) -> Net-(R26-Pad2)
- Q7 pad 3: Net-(Q7-Pad3) -> GND
- Q8 pad 1: +5V -> Net-(U6-Pad12)
- Q8 pad 2: Net-(Q8-Pad2) -> Net-(R27-Pad2)
- Q8 pad 3: Net-(Q8-Pad3) -> GND
- R10 pad 1: /Display_life/D1_CA1 -> Net-(U2-Pad6)
- R10 pad 2: Net-(Q1-Pad3) -> /Display_life/g1
- R11 pad 1: /Display_life/D1_CA2 -> Net-(U2-Pad7)
- R11 pad 2: Net-(Q2-Pad3) -> /Display_life/dp1
- R12 pad 1: /Display_life/D1_CA3 -> Net-(U3-Pad15)
- R12 pad 2: Net-(Q3-Pad3) -> Net-(U6-Pad11)
- R13 pad 1: /Display_life/D1_CA4 -> Net-(U3-Pad1)
- R13 pad 2: Net-(Q4-Pad3) -> Net-(U6-Pad7)
- R14 pad 1: /Display_life/D1_CA5 -> Net-(U3-Pad2)
- R14 pad 2: Net-(Q5-Pad3) -> Net-(U6-Pad4)
- R15 pad 1: GND -> Net-(U3-Pad3)
- R15 pad 2: Net-(R15-Pad2) -> Net-(U6-Pad2)
- R16 pad 1: GND -> Net-(U3-Pad4)
- R16 pad 2: Net-(R16-Pad2) -> Net-(U6-Pad1)
- R17 pad 1: GND -> Net-(U3-Pad5)
- R17 pad 2: Net-(R17-Pad2) -> Net-(U6-Pad10)
- R18 pad 1: GND -> Net-(U3-Pad6)
- R18 pad 2: Net-(R18-Pad2) -> Net-(U6-Pad5)
- R19 pad 1: GND -> Net-(U3-Pad7)
- R19 pad 2: Net-(R19-Pad2) -> Net-(U6-Pad3)
- R2 pad 1: Net-(R2-Pad1) -> Net-(U1-Pad14)
- R2 pad 2: Net-(R2-Pad2) -> /RX
- R20 pad 1: GND -> /Display_life/D1_CA4
- R21 pad 1: GND -> /Display_life/D1_CA3
- R22 pad 1: GND -> /Display_life/D1_CA2
- R23 pad 1: Net-(R23-Pad1) -> /Display_life/D1_CA1
- R24 pad 1: Net-(R24-Pad1) -> /Display_life/D2_CA4
- R25 pad 1: Net-(R25-Pad1) -> /Display_life/D2_CA3
- R26 pad 1: Net-(R26-Pad1) -> /Display_life/D2_CA2
- R27 pad 1: Net-(R27-Pad1) -> /Display_life/D2_CA1
- R28 pad 1: Net-(R28-Pad1) -> GND
- R28 pad 2: Net-(R28-Pad2) -> Net-(SW2-Pad1)
- R29 pad 1: Net-(R29-Pad1) -> GND
- R29 pad 2: Net-(R29-Pad2) -> Net-(SW3-Pad1)
- R3 pad 1: Net-(R3-Pad1) -> Net-(U1-Pad15)
- R3 pad 2: Net-(R3-Pad2) -> /TX
- R30 pad 1: Net-(R30-Pad1) -> GND
- R30 pad 2: Net-(R30-Pad2) -> Net-(SW4-Pad1)
- R31 pad 1: /Display_life/D2_CA1 -> GND
- R31 pad 2: Net-(Q6-Pad3) -> Net-(SW5-Pad1)
- R32 pad 1: /Display_life/D2_CA2 -> GND
- R32 pad 2: Net-(Q7-Pad3) -> Net-(SW6-Pad1)
- R33 pad 1: /Display_life/D2_CA3 -> GND
- R33 pad 2: Net-(Q8-Pad3) -> Net-(SW7-Pad1)
- R34 pad 1: /Display_life/D2_CA4 -> GND
- R34 pad 2: Net-(Q9-Pad3) -> Net-(SW8-Pad1)
- R35 pad 1: /Display_life/D2_CA5 -> GND
- R35 pad 2: Net-(Q10-Pad3) -> Net-(SW9-Pad1)
- R36 pad 2: Net-(R36-Pad2) -> Net-(SW10-Pad1)
- R37 pad 2: Net-(R37-Pad2) -> Net-(SW11-Pad1)
- R38 pad 2: Net-(R38-Pad2) -> Net-(SW12-Pad1)
- R39 pad 2: Net-(R39-Pad2) -> Net-(SW13-Pad1)
- R4 pad 1: Net-(R4-Pad1) -> Net-(U2-Pad15)
- R4 pad 2: Net-(R4-Pad2) -> /Display_life/a1
- R40 pad 2: Net-(R40-Pad2) -> Net-(SW14-Pad1)
- R41 pad 2: Net-(R41-Pad2) -> Net-(SW15-Pad1)
- R42 pad 2: Net-(R42-Pad2) -> Net-(SW16-Pad1)
- R43 pad 2: Net-(R43-Pad2) -> Net-(SW17-Pad1)
- R5 pad 1: Net-(R5-Pad1) -> Net-(U2-Pad1)
- R5 pad 2: Net-(R5-Pad2) -> /Display_life/b1
- R6 pad 1: Net-(R6-Pad1) -> Net-(U2-Pad2)
- R6 pad 2: Net-(R6-Pad2) -> /Display_life/c1
- R7 pad 1: Net-(R7-Pad1) -> Net-(U2-Pad3)
- R7 pad 2: Net-(R7-Pad2) -> /Display_life/d1
- R8 pad 1: Net-(R8-Pad1) -> Net-(U2-Pad4)
- R8 pad 2: Net-(R8-Pad2) -> /Display_life/e1
- R9 pad 1: Net-(R9-Pad1) -> Net-(U2-Pad5)
- R9 pad 2: Net-(R9-Pad2) -> /Display_life/f1
- SW1 pad 1: Net-(R15-Pad2) -> GND
- SW1 pad 2: +5V -> /Reset
- SW10 pad 1: Net-(R37-Pad2) -> Net-(SW10-Pad1)
- SW11 pad 1: Net-(R38-Pad2) -> Net-(SW11-Pad1)
- SW12 pad 1: Net-(R39-Pad2) -> Net-(SW12-Pad1)
- SW13 pad 1: Net-(R40-Pad2) -> Net-(SW13-Pad1)
- SW14 pad 1: Net-(R41-Pad2) -> Net-(SW14-Pad1)
- SW15 pad 1: Net-(R42-Pad2) -> Net-(SW15-Pad1)
- SW16 pad 1: Net-(R43-Pad2) -> Net-(SW16-Pad1)
- SW17 pad 1: Net-(R44-Pad2) -> Net-(SW17-Pad1)
- SW2 pad 1: Net-(R16-Pad2) -> Net-(SW2-Pad1)
- SW3 pad 1: Net-(R17-Pad2) -> Net-(SW3-Pad1)
- SW4 pad 1: Net-(R18-Pad2) -> Net-(SW4-Pad1)
- SW5 pad 1: Net-(R19-Pad2) -> Net-(SW5-Pad1)
- SW6 pad 1: Net-(R20-Pad2) -> Net-(SW6-Pad1)
- SW7 pad 1: Net-(R21-Pad2) -> Net-(SW7-Pad1)
- SW8 pad 1: Net-(R22-Pad2) -> Net-(SW8-Pad1)
- SW9 pad 1: Net-(R36-Pad2) -> Net-(SW9-Pad1)
- U1 pad 1: /PB1 -> /PB0
- U1 pad 14: /PD0 -> Net-(U1-Pad14)
- U1 pad 15: /PD1 -> Net-(U1-Pad15)
- U1 pad 16: /PD2 -> unconnected-(U1-Pad16)
- U1 pad 17: /PD3 -> unconnected-(U1-Pad17)
- U1 pad 2: /PB2 -> /PB1
- U1 pad 22: unconnected-(U1-Pad22) -> /PD0
- U1 pad 23: unconnected-(U1-Pad23) -> /PD1
- U1 pad 24: unconnected-(U1-Pad24) -> /PD2
- U1 pad 25: unconnected-(U1-Pad25) -> /PD3
- U1 pad 3: /PB3 -> /PB2
- U2 pad 1: Net-(R3-Pad1) -> Net-(U2-Pad1)
- U2 pad 11: /PB2 -> /PB1
- U2 pad 12: /PB3 -> /PB2
- U2 pad 14: /PB1 -> /PB0
- U2 pad 15: Net-(R2-Pad1) -> Net-(U2-Pad15)
- U2 pad 2: Net-(R4-Pad1) -> Net-(U2-Pad2)
- U2 pad 3: Net-(R5-Pad1) -> Net-(U2-Pad3)
- U2 pad 4: Net-(R6-Pad1) -> Net-(U2-Pad4)
- U2 pad 5: Net-(R7-Pad1) -> Net-(U2-Pad5)
- U2 pad 6: Net-(R8-Pad1) -> Net-(U2-Pad6)
- U2 pad 7: Net-(R9-Pad1) -> Net-(U2-Pad7)
- U3 pad 1: Net-(R24-Pad1) -> Net-(U3-Pad1)
- U3 pad 11: /PB2 -> /PB1
- U3 pad 12: /PB3 -> /PB2
- U3 pad 15: Net-(R23-Pad1) -> Net-(U3-Pad15)
- U3 pad 2: Net-(R25-Pad1) -> Net-(U3-Pad2)
- U3 pad 3: Net-(R26-Pad1) -> Net-(U3-Pad3)
- U3 pad 4: Net-(R27-Pad1) -> Net-(U3-Pad4)
- U3 pad 5: Net-(R28-Pad1) -> Net-(U3-Pad5)
- U3 pad 6: Net-(R29-Pad1) -> Net-(U3-Pad6)
- U3 pad 7: Net-(R30-Pad1) -> Net-(U3-Pad7)
- U3 pad 9: /next_bitshifter -> unconnected-(U3-Pad9)
- U4 pad 1: /Display_life/D1_CA5 -> unconnected-(U4-Pad1)
- U4 pad 5: /Display_life/D2_CA5 -> unconnected-(U4-Pad5)
- U5 pad 1: Net-(Q1-Pad2) -> /Display_life/e1
- U5 pad 11: Net-(R7-Pad2) -> /Display_life/a1
- U5 pad 2: Net-(Q2-Pad2) -> /Display_life/d1
- U5 pad 3: Net-(R5-Pad2) -> /Display_life/dp1
- U5 pad 4: Net-(Q5-Pad2) -> /Display_life/c1
- U5 pad 5: Net-(R6-Pad2) -> /Display_life/g1
- U5 pad 6: Net-(Q3-Pad2) -> Net-(U5-Pad6)
- U5 pad 7: Net-(R9-Pad2) -> /Display_life/b1
- U5 pad 8: Net-(Q4-Pad2) -> Net-(U5-Pad8)
- U5 pad 9: unconnected-(U5-Pad9) -> Net-(U5-Pad9)
- U6 pad 1: Net-(Q6-Pad2) -> Net-(U6-Pad1)
- U6 pad 11: Net-(R28-Pad2) -> Net-(U6-Pad11)
- U6 pad 2: Net-(Q7-Pad2) -> Net-(U6-Pad2)
- U6 pad 3: Net-(R26-Pad2) -> Net-(U6-Pad3)
- U6 pad 4: Net-(Q10-Pad2) -> Net-(U6-Pad4)
- U6 pad 5: Net-(R27-Pad2) -> Net-(U6-Pad5)
- U6 pad 6: Net-(Q8-Pad2) -> Net-(U6-Pad6)
- U6 pad 7: Net-(R30-Pad2) -> Net-(U6-Pad7)
- U6 pad 8: Net-(Q9-Pad2) -> Net-(U6-Pad8)
- U6 pad 9: unconnected-(U6-Pad9) -> Net-(U6-Pad9)
- U7 pad 11: Net-(R15-Pad2) -> Net-(SW2-Pad1)
- U7 pad 12: Net-(R16-Pad2) -> Net-(SW3-Pad1)
- U7 pad 13: Net-(R17-Pad2) -> Net-(SW4-Pad1)
- U7 pad 14: Net-(R18-Pad2) -> Net-(SW5-Pad1)
- U7 pad 3: Net-(R19-Pad2) -> Net-(SW6-Pad1)
- U7 pad 4: Net-(R20-Pad2) -> Net-(SW7-Pad1)
- U7 pad 5: Net-(R21-Pad2) -> Net-(SW8-Pad1)
- U7 pad 6: Net-(R22-Pad2) -> Net-(SW9-Pad1)
- U8 pad 11: Net-(R36-Pad2) -> Net-(SW10-Pad1)
- U8 pad 12: Net-(R37-Pad2) -> Net-(SW11-Pad1)
- U8 pad 13: Net-(R38-Pad2) -> Net-(SW12-Pad1)
- U8 pad 14: Net-(R39-Pad2) -> Net-(SW13-Pad1)
- U8 pad 3: Net-(R40-Pad2) -> Net-(SW14-Pad1)
- U8 pad 4: Net-(R41-Pad2) -> Net-(SW15-Pad1)
- U8 pad 5: Net-(R42-Pad2) -> Net-(SW16-Pad1)
- U8 pad 6: Net-(R43-Pad2) -> Net-(SW17-Pad1)

Commit message: reduced to 2 displays and logig analyzer output added
Parts:
- added J5: 2nd Bit_shifter, Connector_PinHeader_2.54mm:PinHeader_1x03_P2.54mm_Vertical, F.Cu at (9.38, 132.4)
- added J6: 2nd 7 Segment, Connector_PinHeader_2.54mm:PinHeader_1x08_P2.54mm_Vertical, F.Cu at (0.08, 132.4)
- added J7: decoder_input, Connector_PinHeader_2.54mm:PinHeader_1x04_P2.54mm_Vertical, F.Cu at (55.3, 71.5)
- added J8: disp_1_decoder, Connector_PinHeader_2.54mm:PinHeader_1x04_P2.54mm_Vertical, F.Cu at (70.9, 66.4)
- added J9: disp_2_decoder, Connector_PinHeader_2.54mm:PinHeader_1x04_P2.54mm_Vertical, F.Cu at (55.3, 76.6)
- moved U3 274.2 mm to (-0.45, 119.3)
- moved C10 271.2 mm to (-7.77, 115.8)
- moved C9 271.2 mm to (-7.77, 113.1)
- moved C6 216.0 mm to (60.5, 29.2), turned to 180 degrees
- moved C5 214.4 mm to (63.1, 29.2), turned to 0 degrees
- moved R34 195.2 mm to (122.1, 75.2), turned to 90 degrees
- moved SW2 188.8 mm to (98.1, 56.2)
- moved SW3 188.1 mm to (111.8, 56.2)
- moved SW6 188.1 mm to (98.1, 70.7)
- moved SW4 187.5 mm to (125.6, 56.2)
- moved SW7 187.5 mm to (111.8, 70.7)
- moved SW8 186.8 mm to (125.6, 70.7)
- moved R35 185.7 mm to (135.9, 75.2), turned to 90 degrees
- moved C11 180.0 mm to (95.0, 88.9)
- moved C12 180.0 mm to (95.0, 86.2)
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Connections:
- net Net-(U6-Pad1) renamed /Display_life/e2
- net Net-(U6-Pad10) renamed /Display_life/f2
- net Net-(U6-Pad11) renamed /Display_life/a2
- net Net-(U6-Pad2) renamed /Display_life/d2
- net Net-(U6-Pad3) renamed /Display_life/dp2
- net Net-(U6-Pad4) renamed /Display_life/c2
- net Net-(U6-Pad5) renamed /Display_life/g2
- net Net-(U6-Pad7) renamed /Display_life/b2

Commit message: layout nearly finished and first traces
Parts:
- moved R18 248.8 mm to (70.9, 140.8), turned to 0 degrees
- moved R17 225.0 mm to (81.5, 138.2), turned to 0 degrees
- moved R16 222.2 mm to (70.9, 135.7), turned to 0 degrees
- moved R15 198.4 mm to (81.5, 133.2), turned to 0 degrees
- moved R19 198.2 mm to (81.5, 143.3), turned to 0 degrees
- moved C13 184.9 mm to (58.0, 153.4)
- moved C14 184.9 mm to (58.0, 156.0)
- moved U8 184.2 mm to (62.0, 158.5)
- moved SW14 184.0 mm to (98.1, 165.6)
- moved R36 184.0 mm to (94.6, 158.5)
- moved R40 184.0 mm to (94.6, 170.1)
- moved SW10 183.8 mm to (98.1, 150.9)
- moved SW15 183.4 mm to (111.8, 165.6)
- moved R37 183.4 mm to (108.3, 158.5)
- moved R41 183.4 mm to (108.3, 170.1)
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Routing:
- net /Reset: track 0.00 -> 61.1 mm, vias 0 -> 2
- net /Display_life/c2: track 0.00 -> 48.9 mm
- net /Display_life/g2: track 0.00 -> 48.1 mm
- net Net-(R3-Pad1): track 0.00 -> 47.5 mm, vias 0 -> 1
- net Net-(R2-Pad1): track 0.00 -> 47.0 mm, vias 0 -> 1
- net Net-(C4-Pad1): track 0.00 -> 44.5 mm
- net /Display_life/a2: track 0.00 -> 40.5 mm
- net /Display_life/b2: track 0.00 -> 40.3 mm
- net Net-(C3-Pad1): track 0.00 -> 39.9 mm
- net /Display_life/e2: track 0.00 -> 39.2 mm
- net /Display_life/f2: track 0.00 -> 38.1 mm, vias 0 -> 1
- net /Display_life/dp2: track 0.00 -> 33.6 mm, vias 0 -> 1
- net /Display_life/d2: track 0.00 -> 32.2 mm
- net Net-(Q5-Pad1): track 0.00 -> 25.4 mm
- net Net-(R13-Pad1): track 0.00 -> 24.4 mm
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- added copper zone on F.Cu, net +5V

Commit message: test 1
Connections:
- net /PD0 renamed /PC0
- net /PD1 renamed /PC1
- net /PD2 renamed /PC2
- net /PD3 renamed /PC3
- U8 pad 10: /Buttons_Row_1_and_2/Serial_3 -> unconnected-(U8-Pad10)
Changed lines of the file:
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@@
   (net 20 "unconnected-(U1-Pad29)")
   (net 21 "unconnected-(U1-Pad32)")
-  (net 22 "/PD0")
-  (net 23 "/PD1")
-  (net 24 "/PD2")
-  (net 25 "/PD3")
+  (net 22 "/PC0")
+  (net 23 "/PC1")
+  (net 24 "/PC2")
+  (net 25 "/PC3")
   (net 26 "/PB0")
   (net 27 "/Display_life/dp2")
@@
   (net 56 "Net-(Q2-Pad1)")
   (net 57 "/Buttons_Row_1_and_2/Serial_2")
-  (net 58 "/Buttons_Row_1_and_2/Serial_3")
+  (net 58 "unconnected-(U8-Pad10)")
   (net 59 "Net-(Q2-Pad2)")
   (net 60 "Net-(Q3-Pad1)")
@@
       (net 42 "/PB2") (pinfunction "PB2") (pintype "bidirectional"))
     (pad "4" thru_hole oval (at 0 7.62 90) (size 2.4 1.6) (drill 0.8) (layers *.Cu *.Mask)
-      (net 1 "unconnected-(U1-Pad4)") (pinfunction "PB3") (pintype "bidirectional"))
+      (net 1 "unconnected-(U1-Pad4)") (pinfunction "PB3") (pintype "bidirectional+no_connect"))
     (pad "5" thru_hole oval (at 0 10.16 90) (size 2.4 1.6) (drill 0.8) (layers *.Cu *.Mask)
-      (net 2 "unconnected-(U1-Pad5)") (pinfunction "PB4") (pintype "bidirectional"))
+      (net 2 "unconnected-(U1-Pad5)") (pinfunction "PB4") (pintype "bidirectional+no_connect"))
     (pad "6" thru_hole oval (at 0 12.7 90) (size 2.4 1.6) (drill 0.8) (layers *.Cu *.Mask)
       (net 5 "/MOSI") (pinfunction "PB5") (pintype "bidirectional"))
@@
       (net 73 "Net-(R3-Pad1)") (pinfunction "PD1") (pintype "bidirectional"))
     (pad "16" thru_hole oval (at 0 38.1 90) (size 2.4 1.6) (drill 0.8) (layers *.Cu *.Mask)
-      (net 28 "unconnected-(U1-Pad16)") (pinfunction "PD2") (pintype "bidirectional"))
+      (net 28 "unconnected-(U1-Pad16)") (pinfunction "PD2") (pintype "bidirectional+no_connect"))
     (pad "17" thru_hole oval (at 0 40.64 90) (size 2.4 1.6) (drill 0.8) (layers *.Cu *.Mask)
-      (net 43 "unconnected-(U1-Pad17)") (pinfunction "PD3") (pintype "bidirectional"))
+      (net 43 "unconnected-(U1-Pad17)") (pinfunction "PD3") (pintype "bidirectional+no_connect"))
     (pad "18" thru_hole oval (at 0 43.18 90) (size 2.4 1.6) (drill 0.8) (layers *.Cu *.Mask)
-      (net 7 "unconnected-(U1-Pad18)") (pinfunction "PD4") (pintype "bidirectional"))
+      (net 7 "unconnected-(U1-Pad18)") (pinfunction "PD4") (pintype "bidirectional+no_connect"))
     (pad "19" thru_hole oval (at 0 45.72 90) (size 2.4 1.6) (drill 0.8) (layers *.Cu *.Mask)
-      (net 8 "unconnected-(U1-Pad19)") (pinfunction "PD5") (pintype "bidirectional"))
+      (net 8 "unconnected-(U1-Pad19)") (pinfunction "PD5") (pintype "bidirectional+no_connect"))
     (pad "20" thru_hole oval (at 0 48.26 90) (size 2.4 1.6) (drill 0.8) (layers *.Cu *.Mask)
-      (net 18 "unconnected-(U1-Pad20)") (pinfunction "PD6") (pintype "bidirectional"))
+      (net 18 "unconnected-(U1-Pad20)") (pinfunction "PD6") (pintype "bidirectional+no_connect"))
     (pad "21" thru_hole oval (at 15.24 48.26 90) (size 2.4 1.6) (drill 0.8) (layers *.Cu *.Mask)
-      (net 9 "unconnected-(U1-Pad21)") (pinfunction "PD7") (pintype "bidirectional"))
+      (net 9 "unconnected-(U1-Pad21)") (pinfunction "PD7") (pintype "bidirectional+no_connect"))
     (pad "22" thru_hole oval (at 15.24 45.72 90) (size 2.4 1.6) (drill 0.8) (layers *.Cu *.Mask)
-      (net 22 "/PD0") (pinfunction "PC0") (pintype "bidirectional"))
+      (net 22 "/PC0") (pinfunction "PC0") (pintype "bidirectional"))
     (pad "23" thru_hole oval (at 15.24 43.18 90) (size 2.4 1.6) (drill 0.8) (layers *.Cu *.Mask)
-      (net 23 "/PD1") (pinfunction "PC1") (pintype "bidirectional"))
+      (net 23 "/PC1") (pinfunction "PC1") (pintype "bidirectional"))
     (pad "24" thru_hole oval (at 15.24 40.64 90) (size 2.4 1.6) (drill 0.8) (layers *.Cu *.Mask)
-      (net 24 "/PD2") (pinfunction "PC2") (pintype "bidirectional"))
+      (net 24 "/PC2") (pinfunction "PC2") (pintype "bidirectional"))
     (pad "25" thru_hole oval (at 15.24 38.1 90) (size 2.4 1.6) (drill 0.8) (layers *.Cu *.Mask)
-      (net 25 "/PD3") (pinfunction "PC3") (pintype "bidirectional"))
+      (net 25 "/PC3") (pinfunction "PC3") (pintype "bidirectional"))
     (pad "26" thru_hole oval (at 15.24 35.56 90) (size 2.4 1.6) (drill 0.8) (layers *.Cu *.Mask)
-      (net 13 "unconnected-(U1-Pad26)") (pinfunction "PC4") (pintype "bidirectional"))
+      (net 13 "unconnected-(U1-Pad26)") (pinfunction "PC4") (pintype "bidirectional+no_connect"))
     (pad "27" thru_hole oval (at 15.24 33.02 90) (size 2.4 1.6) (drill 0.8) (layers *.Cu *.Mask)
-      (net 14 "unconnected-(U1-Pad27)") (pinfunction "PC5") (pintype "bidirectional"))
+      (net 14 "unconnected-(U1-Pad27)") (pinfunction "PC5") (pintype "bidirectional+no_connect"))
     (pad "28" thru_hole oval (at 15.24 30.48 90) (size 2.4 1.6) (drill 0.8) (layers *.Cu *.Mask)
-      (net 15 "unconnected-(U1-Pad28)") (pinfunction "PC6") (pintype "bidirectional"))
+      (net 15 "unconnected-(U1-Pad28)") (pinfunction "PC6") (pintype "bidirectional+no_connect"))
     (pad "29" thru_hole oval (at 15.24 27.94 90) (size 2.4 1.6) (drill 0.8) (layers *.Cu *.Mask)
-      (net 20 "unconnected-(U1-Pad29)") (pinfunction "PC7") (pintype "bidirectional"))
+      (net 20 "unconnected-(U1-Pad29)") (pinfunction "PC7") (pintype "bidirectional+no_connect"))
     (pad "30" thru_hole oval (at 15.24 25.4 90) (size 2.4 1.6) (drill 0.8) (layers *.Cu *.Mask)
       (net 16 "+5V") (pinfunction "AVCC") (pintype "power_in"))
@@
       (net 17 "GND") (pinfunction "GND") (pintype "passive"))
     (pad "32" thru_hole oval (at 15.24 20.32 90) (size 2.4 1.6) (drill 0.8) (layers *.Cu *.Mask)
-      (net 21 "unconnected-(U1-Pad32)") (pinfunction "AREF") (pintype "passive"))
+      (net 21 "unconnected-(U1-Pad32)") (pinfunction "AREF") (pintype "passive+no_connect"))
     (pad "33" thru_hole oval (at 15.24 17.78 90) (size 2.4 1.6) (drill 0.8) (layers *.Cu *.Mask)
       (net 114 "/PA7") (pinfunction "PA7") (pintype "bidirectional"))
@@
     (fp_line (start 6.985 -1.27) (end 6.985 19.05) (layer "F.Fab") (width 0.1))
     (pad "1" thru_hole oval (at 0 0 90) (size 2.4 1.6) (drill 0.8) (layers *.Cu *.Mask)
-      (net 23 "/PD1") (pinfunction "~{PL}") (pintype "input"))
+      (net 23 "/PC1") (pinfunction "~{PL}") (pintype "input"))
     (pad "2" thru_hole oval (at 0 2.54 90) (size 2.4 1.6) (drill 0.8) (layers *.Cu *.Mask)
-      (net 22 "/PD0") (pinfunction "CP") (pintype "input"))
+      (net 22 "/PC0") (pinfunction "CP") (pintype "input"))
     (pad "3" thru_hole oval (at 0 5.08 90) (size 2.4 1.6) (drill 0.8) (layers *.Cu *.Mask)
       (net 94 "Net-(R32-Pad2)") (pinfunction "D4") (pintype "input"))
@@
       (net 17 "GND") (pinfunction "GND") (pintype "power_in"))
     (pad "9" thru_hole oval (at 7.62 17.78 90) (size 2.4 1.6) (drill 0.8) (layers *.Cu *.Mask)
-      (net 25 "/PD3") (pinfunction "Q7") (pintype "output"))
+      (net 25 "/PC3") (pinfunction "Q7") (pintype "output"))
     (pad "10" thru_hole oval (at 7.62 15.24 90) (size 2.4 1.6) (drill 0.8) (layers *.Cu *.Mask)
       (net 57 "/Buttons_Row_1_and_2/Serial_2") (pinfunction "DS") (pintype "input"))
@@
       (net 93 "Net-(R31-Pad2)") (pinfunction "D3") (pintype "input"))
     (pad "15" thru_hole oval (at 7.62 2.54 90) (size 2.4 1.6) (drill 0.8) (layers *.Cu *.Mask)
-      (net 24 "/PD2") (pinfunction "~{CE}") (pintype "input"))
+      (net 24 "/PC2") (pinfunction "~{CE}") (pintype "input"))
     (pad "16" thru_hole oval (at 7.62 0 90) (size 2.4 1.6) (drill 0.8) (layers *.Cu *.Mask)
       (net 16 "+5V") (pinfunction "VCC") (pintype "power_in"))
@@
     (fp_line (start 6.985 19.05) (end 0.635 19.05) (layer "F.Fab") (width 0.1))
     (pad "1" thru_hole oval (at 0 0 90) (size 2.4 1.6) (drill 0.8) (layers *.Cu *.Mask)
-      (net 23 "/PD1") (pinfunction "~{PL}") (pintype "input"))
+      (net 23 "/PC1") (pinfunction "~{PL}") (pintype "input"))
     (pad "2" thru_hole oval (at 0 2.54 90) (size 2.4 1.6) (drill 0.8) (layers *.Cu *.Mask)
-      (net 22 "/PD0") (pinfunction "CP") (pintype "input"))
+      (net 22 "/PC0") (pinfunction "CP") (pintype "input"))
     (pad "3" thru_hole oval (at 0 5.08 90) (size 2.4 1.6) (drill 0.8) (layers *.Cu *.Mask)
       (net 102 "Net-(R40-Pad2)") (pinfunction "D4") (pintype "input"))
@@
       (net 57 "/Buttons_Row_1_and_2/Serial_2") (pinfunction "Q7") (pintype "output"))
     (pad "10" thru_hole oval (at 7.62 15.24 90) (size 2.4 1.6) (drill 0.8) (layers *.Cu *.Mask)
-      (net 58 "/Buttons_Row_1_and_2/Serial_3") (pinfunction "DS") (pintype "input"))
+      (net 58 "unconnected-(U8-Pad10)") (pinfunction "DS") (pintype "input+no_connect"))
     (pad "11" thru_hole oval (at 7.62 12.7 90) (size 2.4 1.6) (drill 0.8) (layers *.Cu *.Mask)
       (net 98 "Net-(R36-Pad2)") (pinfunction "D0") (pintype "input"))
@@
       (net 101 "Net-(R39-Pad2)") (pinfunction "D3") (pintype "input"))
     (pad "15" thru_hole oval (at 7.62 2.54 90) (size 2.4 1.6) (drill 0.8) (layers *.Cu *.Mask)
-      (net 24 "/PD2") (pinfunction "~{CE}") (pintype "input"))
+      (net 24 "/PC2") (pinfunction "~{CE}") (pintype "input"))
     (pad "16" thru_hole oval (at 7.62 0 90) (size 2.4 1.6) (drill 0.8) (layers *.Cu *.Mask)
       (net 16 "+5V") (pinfunction "VCC") (pintype "power_in"))
