File: pcb/magic_counter.kicad_pcb (KiCad board)
At the start: 2 copper layers, 127.4 x 202.4 mm, 104 parts, among them J1 ISP-Port, J2 Serial Out, J3 1st Bit_shifter, J4 1st 7 Segment, J5 2nd Bit_shifter, J6 2nd 7 Segment, J7 decoder_input, J8 disp_1_decoder, J9 disp_2_decoder, Q1 Q_NPN_CBE, Q2 Q_NPN_CBE, Q3 Q_NPN_CBE, Q4 Q_NPN_CBE, Q5 Q_NPN_CBE, Q6 Q_NPN_CBE, Q7 Q_NPN_CBE, Q8 Q_NPN_CBE, SW1 Random, SW10 Reset, SW11 +1, SW12 +10, SW13 -10, SW14 -1, SW15 x2, SW16 /2, SW17 Random, SW2 Reset, SW3 +1, SW4 +10, SW5 -10, SW6 -1, SW7 x2, SW8 /2, SW9 Random, U1 ATmega32A-P, U2 74HC595, U3 74HC595, U4 4028, U5 CC56-12SURKWA, U6 CC56-12SURKWA, U7 74HC165, U8 74HC165, Y1 Crystal

Commit message: new parts and stuff
Parts:
- added C15: 100pF, Capacitor_THT:C_Disc_D3.8mm_W2.6mm_P2.50mm, F.Cu at (58.0, 168.0)
- added C16: 1nF, Capacitor_THT:C_Disc_D3.8mm_W2.6mm_P2.50mm, F.Cu at (58.0, 171.0)
- added C17: 100pF, Capacitor_THT:C_Disc_D3.8mm_W2.6mm_P2.50mm, F.Cu at (58.0, 180.7)
- added C18: 1nF, Capacitor_THT:C_Disc_D3.8mm_W2.6mm_P2.50mm, F.Cu at (58.0, 183.3)
- added C19: 100pF, Capacitor_THT:C_Disc_D3.8mm_W2.6mm_P2.50mm, F.Cu at (94.1, 180.7)
- added C20: 1nF, Capacitor_THT:C_Disc_D3.8mm_W2.6mm_P2.50mm, F.Cu at (94.1, 183.3)
- added D1: LED, LED_THT:LED_D5.0mm, F.Cu at (45.5, 72.7)
- added D10: LED, LED_THT:LED_D5.0mm, F.Cu at (45.5, 174.5)
- added D11: LED, LED_THT:LED_D5.0mm, F.Cu at (45.5, 185.8)
- added D12: LED, LED_THT:LED_D5.0mm, F.Cu at (45.5, 197.2)
- added D2: LED, LED_THT:LED_D5.0mm, F.Cu at (45.5, 84.0)
- added D3: LED, LED_THT:LED_D5.0mm, F.Cu at (45.5, 95.3)
- added D4: LED, LED_THT:LED_D5.0mm, F.Cu at (45.5, 106.6)
- added D5: LED, LED_THT:LED_D5.0mm, F.Cu at (45.5, 118.0)
- added D6: LED, LED_THT:LED_D5.0mm, F.Cu at (45.5, 129.3)
- added D7: LED, LED_THT:LED_D5.0mm, F.Cu at (45.5, 140.6)
- added D8: LED, LED_THT:LED_D5.0mm, F.Cu at (45.5, 151.9)
- added D9: LED, LED_THT:LED_D5.0mm, F.Cu at (45.5, 163.2)
- added J10: Barrel_Jack_Switch, Connector_BarrelJack:BarrelJack_Horizontal, F.Cu at (45.7, 56.7)
- added J11: Screw_Terminal_01x02, TerminalBlock_Phoenix:TerminalBlock_Phoenix_PT-1,5-2-3.5-H_1x02_P3.50mm_Horizontal, F.Cu at (36.7, 42.9)
- added J12: Conn_01x07_Male, Connector_PinHeader_2.54mm:PinHeader_1x07_P2.54mm_Vertical, F.Cu at (53.8, 143.3)
- added J13: Conn_01x06_Male, Connector_PinHeader_2.54mm:PinHeader_1x06_P2.54mm_Vertical, F.Cu at (86.9, 173.2)
- added R44: 90R, Resistor_THT:R_Axial_DIN0207_L6.3mm_D2.5mm_P7.62mm_Horizontal, F.Cu at (40.5, 72.7)
- added R45: 90R, Resistor_THT:R_Axial_DIN0207_L6.3mm_D2.5mm_P7.62mm_Horizontal, F.Cu at (40.5, 84.0)
- added R46: 90R, Resistor_THT:R_Axial_DIN0207_L6.3mm_D2.5mm_P7.62mm_Horizontal, F.Cu at (40.5, 95.3)
- added R47: 90R, Resistor_THT:R_Axial_DIN0207_L6.3mm_D2.5mm_P7.62mm_Horizontal, F.Cu at (40.5, 106.6)
- added R48: 90R, Resistor_THT:R_Axial_DIN0207_L6.3mm_D2.5mm_P7.62mm_Horizontal, F.Cu at (40.5, 118.0)
- added R49: 90R, Resistor_THT:R_Axial_DIN0207_L6.3mm_D2.5mm_P7.62mm_Horizontal, F.Cu at (40.5, 129.3)
- added R50: 90R, Resistor_THT:R_Axial_DIN0207_L6.3mm_D2.5mm_P7.62mm_Horizontal, F.Cu at (40.5, 140.6)
- added R51: 90R, Resistor_THT:R_Axial_DIN0207_L6.3mm_D2.5mm_P7.62mm_Horizontal, F.Cu at (40.5, 151.9)
- added R52: 90R, Resistor_THT:R_Axial_DIN0207_L6.3mm_D2.5mm_P7.62mm_Horizontal, F.Cu at (40.5, 163.2)
- added R53: 90R, Resistor_THT:R_Axial_DIN0207_L6.3mm_D2.5mm_P7.62mm_Horizontal, F.Cu at (40.5, 174.5)
- added R54: 90R, Resistor_THT:R_Axial_DIN0207_L6.3mm_D2.5mm_P7.62mm_Horizontal, F.Cu at (40.5, 185.8)
- added R55: 90R, Resistor_THT:R_Axial_DIN0207_L6.3mm_D2.5mm_P7.62mm_Horizontal, F.Cu at (40.5, 197.2)
- added R56: 10k, Resistor_THT:R_Axial_DIN0207_L6.3mm_D2.5mm_P7.62mm_Horizontal, F.Cu at (57.3, 204.8)
- added R57: 10k, Resistor_THT:R_Axial_DIN0207_L6.3mm_D2.5mm_P7.62mm_Horizontal, F.Cu at (70.4, 204.8)
- added R58: 10k, Resistor_THT:R_Axial_DIN0207_L6.3mm_D2.5mm_P7.62mm_Horizontal, F.Cu at (83.5, 204.8)
- added R59: 10k, Resistor_THT:R_Axial_DIN0207_L6.3mm_D2.5mm_P7.62mm_Horizontal, F.Cu at (96.6, 204.8)
- added R60: 10k, Resistor_THT:R_Axial_DIN0207_L6.3mm_D2.5mm_P7.62mm_Horizontal, F.Cu at (109.7, 204.8)
- added R61: 10k, Resistor_THT:R_Axial_DIN0207_L6.3mm_D2.5mm_P7.62mm_Horizontal, F.Cu at (122.8, 204.8)
- added R62: 10k, Resistor_THT:R_Axial_DIN0207_L6.3mm_D2.5mm_P7.62mm_Horizontal, F.Cu at (135.9, 204.8)
- added R63: 10k, Resistor_THT:R_Axial_DIN0207_L6.3mm_D2.5mm_P7.62mm_Horizontal, F.Cu at (149.0, 204.8)
- added SW18: Reset, Button_Switch_THT:SW_PUSH_6mm_H5mm, F.Cu at (64.4, 197.2)
- added SW19: +1, Button_Switch_THT:SW_PUSH_6mm_H5mm, F.Cu at (77.5, 197.2)
- added SW20: +10, Button_Switch_THT:SW_PUSH_6mm_H5mm, F.Cu at (90.6, 197.2)
- added SW21: -10, Button_Switch_THT:SW_PUSH_6mm_H5mm, F.Cu at (103.7, 197.2)
- added SW22: -1, Button_Switch_THT:SW_PUSH_6mm_H5mm, F.Cu at (116.8, 197.2)
- added SW23: x2, Button_Switch_THT:SW_PUSH_6mm_H5mm, F.Cu at (129.9, 197.2)
- added SW24: /2, Button_Switch_THT:SW_PUSH_6mm_H5mm, F.Cu at (143.0, 197.2)
- added SW25: Random, Button_Switch_THT:SW_PUSH_6mm_H5mm, F.Cu at (156.1, 197.2)
- added U10: 74HC595, Package_DIP:DIP-16_W7.62mm_LongPads, F.Cu at (62.0, 185.8)
- added U11: 74HC165, Package_DIP:DIP-16_W7.62mm_LongPads, F.Cu at (98.1, 185.8)
- added U9: 74HC595, Package_DIP:DIP-16_W7.62mm_LongPads, F.Cu at (62.0, 173.2)
- J4, J6: footprint Connector_PinHeader_2.54mm:PinHeader_1x08_P2.54mm_Vertical -> Connector_PinHeader_2.54mm:PinHeader_1x10_P2.54mm_Vertical
- moved J4 20.3 mm to (92.6, 28.1), turned to 0 degrees
- moved J6 20.3 mm to (92.6, 123.0), turned to 0 degrees
Connections:
- J4 pad 1: /Display_life/dp1 -> +5V
- J4 pad 2: /Display_life/g1 -> /Display_life/a1
- J4 pad 3: /Display_life/f1 -> /Display_life/b1
- J4 pad 4: /Display_life/e1 -> /Display_life/c1
- J4 pad 6: /Display_life/c1 -> /Display_life/e1
- J4 pad 7: /Display_life/b1 -> /Display_life/f1
- J4 pad 8: /Display_life/a1 -> /Display_life/g1
- J6 pad 1: /Display_life/dp2 -> +5V
- J6 pad 2: /Display_life/g2 -> /Display_life/a2
- J6 pad 3: /Display_life/f2 -> /Display_life/b2
- J6 pad 4: /Display_life/e2 -> /Display_life/c2
- J6 pad 6: /Display_life/c2 -> /Display_life/e2
- J6 pad 7: /Display_life/b2 -> /Display_life/f2
- J6 pad 8: /Display_life/a2 -> /Display_life/g2
- U1 pad 18: unconnected-(U1-Pad18) -> /PD4
- U1 pad 19: unconnected-(U1-Pad19) -> /PD5
- U1 pad 20: unconnected-(U1-Pad20) -> /PD6
- U1 pad 26: unconnected-(U1-Pad26) -> /PC4
- U1 pad 27: unconnected-(U1-Pad27) -> /PC5
- U1 pad 28: unconnected-(U1-Pad28) -> /PC6
- U1 pad 29: unconnected-(U1-Pad29) -> /PC7
- U1 pad 33: /PA7 -> unconnected-(U1-Pad33)
- U1 pad 34: /PA6 -> unconnected-(U1-Pad34)
- U1 pad 35: /PA5 -> unconnected-(U1-Pad35)
- U1 pad 36: /PA4 -> unconnected-(U1-Pad36)
Routing:
- net GND: track 0.00 -> 363.8 mm, vias 0 -> 6
- net +5V: track 5.04 -> 287.0 mm, vias 0 -> 4
- net /PC0: track 0.00 -> 209.3 mm, vias 0 -> 1
- net /PC1: track 0.00 -> 208.4 mm, vias 0 -> 1
- net /PC2: track 0.00 -> 199.5 mm, vias 0 -> 2
- net /PD4: track 0.00 -> 197.6 mm
- net /PD6: track 0.00 -> 180.2 mm, vias 0 -> 1
- net /Buttons_Row_1_and_2/Serial_2: track 0.00 -> 178.1 mm
- net /PD5: track 0.00 -> 174.9 mm, vias 0 -> 1
- net /PC4: track 0.00 -> 156.0 mm, vias 0 -> 2
- net /PC6: track 0.00 -> 155.1 mm, vias 0 -> 1
- net /PB2: track 11.0 -> 166.0 mm, vias 0 -> 2
- net /PC5: track 0.00 -> 154.9 mm, vias 0 -> 1
- net /PB1: track 7.42 -> 162.2 mm, vias 0 -> 1
- net /PC7: track 0.00 -> 139.3 mm, vias 0 -> 1
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Other:
- board text added: "5V"
- board text added: "A"
- board text added: "Attack"
- board text added: "B"
- board text added: "Block"
- board text added: "C"
- board text added: "D"
- board text added: "DP"
- board text added: "Damage"
- board text added: "Draw"
- board text added: "E"
- board text added: "End"
- board text added: "End Combat"
- board text added: "F"
- board text added: "G"
- board text added: "GND"
- board text added: "Main 1"
- board text added: "Main 2"
- board text added: "Pass/ Next"
- board text added: "RX"
- board text added: "Start Combat"
- board text added: "TX"
- board text added: "Untap"
- board text added: "Upkeep"

Commit message: finish layout
Other:
- board text added: "+1"
- board text added: "+10"
- board text added: "-1"
- board text added: "-10"
- board text added: "/2"
- board text added: "Add Counter"
- board text added: "Add Player"
- board text added: "Next Display"
- board text added: "Next Phase"
- board text added: "Phases off"
- board text added: "Previous Display"
- board text added: "Previous Phase"
- board text added: "Random"
- board text added: "Remove Counter"
- board text added: "Reset"
- board text added: "x2"
Changed lines of the file:
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@@
       (layerselection 0x00010fc_ffffffff)
       (disableapertmacros false)
-      (usegerberextensions false)
-      (usegerberattributes true)
-      (usegerberadvancedattributes true)
-      (creategerberjobfile true)
+      (usegerberextensions true)
+      (usegerberattributes false)
+      (usegerberadvancedattributes false)
+      (creategerberjobfile false)
       (svguseinch false)
       (svgprecision 6)
@@
       (psa4output false)
       (plotreference true)
-      (plotvalue true)
+      (plotvalue false)
       (plotinvisibletext false)
       (sketchpadsonfab false)
-      (subtractmaskfromsilk false)
+      (subtractmaskfromsilk true)
       (outputformat 1)
       (mirror false)
-      (drillshape 1)
+      (drillshape 0)
       (scaleselection 1)
-      (outputdirectory "")
+      (outputdirectory "gerber/")
     )
   )
@@
     (property "Sheetname" "Phase Switch")
     (attr through_hole)
-    (fp_text reference "SW19" (at 3.25 -2) (layer "F.SilkS")
+    (fp_text reference "SW19" (at 4.5 7.5) (layer "F.SilkS")
       (effects (font (size 1 1) (thickness 0.15)))
     )
@@
     (property "Sheetname" "Phase Switch")
     (attr through_hole)
-    (fp_text reference "SW25" (at 3.25 -2) (layer "F.SilkS")
+    (fp_text reference "SW25" (at 4.5 7.5) (layer "F.SilkS")
       (effects (font (size 1 1) (thickness 0.15)))
     )
@@
     (property "Sheetname" "Phase Switch")
     (attr through_hole)
-    (fp_text reference "SW21" (at 3.25 -2) (layer "F.SilkS")
+    (fp_text reference "SW21" (at 4.5 7.5) (layer "F.SilkS")
       (effects (font (size 1 1) (thickness 0.15)))
     )
@@
     (property "Sheetname" "Phase Switch")
     (attr through_hole)
-    (fp_text reference "SW24" (at 3.25 -2) (layer "F.SilkS")
+    (fp_text reference "SW24" (at 4.5 7.5) (layer "F.SilkS")
       (effects (font (size 1 1) (thickness 0.15)))
     )
@@
     (property "Sheetname" "Phase Switch")
     (attr through_hole)
-    (fp_text reference "SW18" (at 3.25 -2) (layer "F.SilkS")
+    (fp_text reference "SW18" (at 4.5 7.5) (layer "F.SilkS")
       (effects (font (size 1 1) (thickness 0.15)))
     )
@@
     (property "Sheetname" "Phase Switch")
     (attr through_hole)
-    (fp_text reference "SW23" (at 3.25 -2) (layer "F.SilkS")
+    (fp_text reference "SW23" (at 4.5 7.5) (layer "F.SilkS")
       (effects (font (size 1 1) (thickness 0.15)))
     )
@@
     (property "Sheetname" "Phase Switch")
     (attr through_hole)
-    (fp_text reference "SW22" (at 3.25 -2) (layer "F.SilkS")
+    (fp_text reference "SW22" (at 4.5 7.5) (layer "F.SilkS")
       (effects (font (size 1 1) (thickness 0.15)))
     )
@@
     (fp_line (start -2.18 -5.1) (end 5.72 -5.1) (layer "F.Fab") (width 0.1))
     (fp_line (start 4.52 -3.91) (end 4.52 8.99) (layer "F.Fab") (width 0.1))
-    (pad "1" thru_hole roundrect (at 0 0 90) (size 1.7 1.7) (drill 1) (layers *.Cu *.Mask) (roundrect_rratio 0.147059)
+    (pad "1" thru_hole roundrect (at 0 0 90) (size 1.7 1.7) (drill 1) (layers *.Cu *.Mask) (roundrect_rratio 0.1470588235)
       (net 3 "/MISO") (pinfunction "Pin_1") (pintype "passive"))
     (pad "2" thru_hole circle (at 2.54 0 90) (size 1.7 1.7) (drill 1) (layers *.Cu *.Mask)
@@
     (property "Sheetname" "Phase Switch")
     (attr through_hole)
-    (fp_text reference "SW20" (at 3.25 -2) (layer "F.SilkS")
+    (fp_text reference "SW20" (at 4.5 7.5) (layer "F.SilkS")
       (effects (font (size 1 1) (thickness 0.15)))
     )
@@
     (effects (font (size 1 1) (thickness 0.15)))
   )
+  (gr_text "-10" (at 115.076666 162.4875) (layer "F.SilkS")
+    (effects (font (size 1.5 1.5) (thickness 0.3)))
+  )
+  (gr_text "Next\nDisplay" (at 139.75 201.0835) (layer "F.SilkS")
+    (effects (font (size 1.5 1.5) (thickness 0.3)))
+  )
   (gr_text "Main 1" (at 46.73 101.61) (layer "F.SilkS")
     (effects (font (size 1.5 1.5) (thickness 0.3)))
@@
     (effects (font (size 1.5 1.5) (thickness 0.3)))
   )
+  (gr_text "+1" (at 101.31 63.6125) (layer "F.SilkS")
+    (effects (font (size 1.5 1.5) (thickness 0.3)))
+  )
   (gr_text "End\nCombat" (at 46.73 157.58) (layer "F.SilkS")
     (effects (font (size 1.5 1.5) (thickness 0.3)))
@@
     (effects (font (size 1.5 1.5) (thickness 0.3)))
   )
+  (gr_text "+10" (at 115.076666 63.6125) (layer "F.SilkS")
+    (effects (font (size 1.5 1.5) (thickness 0.3)))
+  )
+  (gr_text "x2" (at 128.843332 158.4875) (layer "F.SilkS")
+    (effects (font (size 1.5 1.5) (thickness 0.3)))
+  )
   (gr_text "GND" (at 95.58 145.8675) (layer "F.SilkS")
     (effects (font (size 1 1) (thickness 0.15)))
@@
     (effects (font (size 1 1) (thickness 0.15)))
   )
+  (gr_text "+10" (at 115.076666 158.4875) (layer "F.SilkS")
+    (effects (font (size 1.5 1.5) (thickness 0.3)))
+  )
   (gr_text "C" (at 95.58 130.6275) (layer "F.SilkS")
     (effects (font (size 1 1) (thickness 0.15)))
   )
+  (gr_text "+1" (at 101.31 158.4875) (layer "F.SilkS")
+    (effects (font (size 1.5 1.5) (thickness 0.3)))
+  )
   (gr_text "Attack" (at 46.73 123.658324) (layer "F.SilkS")
     (effects (font (size 1.5 1.5) (thickness 0.3)))
@@
     (effects (font (size 1 1) (thickness 0.15)))
   )
+  (gr_text "/2" (at 128.843332 67.6) (layer "F.SilkS")
+    (effects (font (size 1.5 1.5) (thickness 0.3)))
+  )
+  (gr_text "Previous\nPhase" (at 74.25 201.0835) (layer "F.SilkS")
+    (effects (font (size 1.5 1.5) (thickness 0.3)))
+  )
+  (gr_text "Reset" (at 142.61 63.6125) (layer "F.SilkS")
+    (effects (font (size 1.5 1.5) (thickness 0.3)))
+  )
   (gr_text "End" (at 46.73 180.64) (layer "F.SilkS")
     (effects (font (size 1.5 1.5) (thickness 0.3)))
@@
     (effects (font (size 1 1) (thickness 0.15)))
   )
+  (gr_text "x2" (at 128.843332 63.6125) (layer "F.SilkS")
+    (effects (font (size 1.5 1.5) (thickness 0.3)))
+  )
+  (gr_text "Add\nPlayer" (at 100.45 201.0835) (layer "F.SilkS")
+    (effects (font (size 1.5 1.5) (thickness 0.3)))
+  )
   (gr_text "F" (at 95.58 138.2475) (layer "F.SilkS")
     (effects (font (size 1 1) (thickness 0.15)))
@@
     (effects (font (size 1 1) (thickness 0.15)))
   )
+  (gr_text "Add\nCounter" (at 113.55 201.0835) (layer "F.SilkS")
+    (effects (font (size 1.5 1.5) (thickness 0.3)))
+  )
   (gr_text "TX" (at 68.535 111.03) (layer "F.SilkS")
     (effects (font (size 1 1) (thickness 0.15)))
   )
+  (gr_text "Previous\nDisplay" (at 152.85 201.0835) (layer "F.SilkS")
+    (effects (font (size 1.5 1.5) (thickness 0.3)))
+  )
   (gr_text "GND" (at 73.615 111.03) (layer "F.SilkS")
     (effects (font (size 1 1) (thickness 0.15)))
@@
     (effects (font (size 1.5 1.5) (thickness 0.3)))
   )
+  (gr_text "Random" (at 142.61 67.6) (layer "F.SilkS")
+    (effects (font (size 1.5 1.5) (thickness 0.3)))
+  )
   (gr_text "5V" (at 95.58 28.1325) (layer "F.SilkS")
     (effects (font (size 1 1) (thickness 0.15)))
   )
+  (gr_text "Remove\nCounter" (at 126.65 201.0835) (layer "F.SilkS")
+    (effects (font (size 1.5 1.5) (thickness 0.3)))
+  )
   (gr_text "Damage" (at 46.73 146.53) (layer "F.SilkS")
     (effects (font (size 1.5 1.5) (thickness 0.3)))
   )
+  (gr_text "Next\nPhase" (at 61.15 201.0835) (layer "F.SilkS")
+    (effects (font (size 1.5 1.5) (thickness 0.3)))
+  )
+  (gr_text "-10" (at 115.076666 67.6) (layer "F.SilkS")
+    (effects (font (size 1.5 1.5) (thickness 0.3)))
+  )
   (gr_text "B" (at 95.58 33.2125) (layer "F.SilkS")
     (effects (font (size 1 1) (thickness 0.15)))
   )
+  (gr_text "Random" (at 142.61 162.4875) (layer "F.SilkS")
+    (effects (font (size 1.5 1.5) (thickness 0.3)))
+  )
   (gr_text "D" (at 95.58 133.1675) (layer "F.SilkS")
     (effects (font (size 1 1) (thickness 0.15)))
@@
     (effects (font (size 1 1) (thickness 0.15)))
   )
+  (gr_text "-1" (at 101.31 67.6) (layer "F.SilkS")
+    (effects (font (size 1.5 1.5) (thickness 0.3)))
+  )
+  (gr_text "Phases\noff" (at 87.35 201.0835) (layer "F.SilkS")
+    (effects (font (size 1.5 1.5) (thickness 0.3)))
+  )
   (gr_text "E" (at 95.58 40.8325) (layer "F.SilkS")
     (effects (font (size 1 1) (thickness 0.15)))
   )
+  (gr_text "-1" (at 101.31 162.4875) (layer "F.SilkS")
+    (effects (font (size 1.5 1.5) (thickness 0.3)))
+  )
+  (gr_text "/2" (at 128.843332 162.4875) (layer "F.SilkS")
+    (effects (font (size 1.5 1.5) (thickness 0.3)))
+  )
+  (gr_text "Reset" (at 83.805 90.4) (layer "F.SilkS")
+    (effects (font (size 1.5 1.5) (thickness 0.3)))
+  )
   (gr_text "Upkeep" (at 46.73 78.35025) (layer "F.SilkS")
     (effects (font (size 1.5 1.5) (thickness 0.3)))
@@
     (effects (font (size 1 1) (thickness 0.15)))
   )
+  (gr_text "Reset" (at 142.61 158.4875) (layer "F.SilkS")
+    (effects (font (size 1.5 1.5) (thickness 0.3)))
+  )
   (gr_text "RX" (at 71.075 111.03) (layer "F.SilkS")

Commit message: new routes
Parts:
- moved J12 99.8 mm to (136.8, 87.8), turned to -90 degrees
- moved J5 30.8 mm to (58.0, 118.0)
- moved J3 25.2 mm to (47.9, 40.8)
- moved R2 5.08 mm to (73.6, 103.6)
- moved R3 5.00 mm to (73.6, 98.5)
Connections:
- J2 pad 2: /RX -> /TX
- J2 pad 3: /TX -> /RX
Routing:
- net GND: track 363.8 -> 92.0 mm, vias 6 -> 0
- net /PC0: track 209.3 -> 34.0 mm, vias 1 -> 0
- net /PC1: track 208.4 -> 35.8 mm, vias 1 -> 0
- net +5V: track 287.0 -> 117.5 mm, vias 4 -> 1
- net /Buttons_Row_1_and_2/Serial_2: track 178.1 -> 29.3 mm
- net /PC2: track 199.5 -> 53.4 mm, vias 2 -> 0
- net /PC3: track 109.2 -> 20.8 mm, vias 3 -> 0
- net Net-(Q4-Pad1): track 46.7 -> 89.1 mm, vias 0 -> 1
- net /PD4: track 197.6 -> 159.9 mm
- net Net-(Q3-Pad1): track 57.5 -> 93.4 mm, vias 0 -> 1
- net /PB2: track 166.0 -> 153.0 mm, vias 2 -> 0
- net /Display_life/2nd_Bitshifter: track 111.2 -> 98.4 mm
- net /MOSI: track 42.5 -> 53.3 mm, vias 1 -> 0
- net /PD5: track 174.9 -> 164.2 mm, vias 1 -> 0
- net /PB0: track 121.4 -> 113.0 mm
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