File: pcb/magic_counter.kicad_pcb (KiCad board)
At the start: 2 copper layers, 127.4 x 202.4 mm, 157 parts, among them J1 ISP-Port, J10 Barrel_Jack_Switch, J11 Screw_Terminal_01x02, J12 Conn_01x07_Male, J13 Conn_01x06_Male, J2 Serial Out, J3 1st Bit_shifter, J4 1st 7 Segment, J5 2nd Bit_shifter, J6 2nd 7 Segment, J7 decoder_input, J8 disp_1_decoder, J9 disp_2_decoder, Q1 Q_NPN_CBE, Q2 Q_NPN_CBE, Q3 Q_NPN_CBE, Q4 Q_NPN_CBE, Q5 Q_NPN_CBE, Q6 Q_NPN_CBE, Q7 Q_NPN_CBE, Q8 Q_NPN_CBE, SW1 Random, SW10 Reset, SW11 +1, SW12 +10, SW13 -10, SW14 -1, SW15 x2, SW16 /2, SW17 Random, SW18 Reset, SW19 +1, SW2 Reset, SW20 +10, SW21 -10, SW22 -1, SW23 x2, SW24 /2, SW25 Random, SW3 +1, SW4 +10, SW5 -10, SW6 -1, SW7 x2, SW8 /2, SW9 Random, U1 ATmega32A-P, U10 74HC595, U11 74HC165, U2 74HC595, U3 74HC595, U4 4028, U5 CC56-12SURKWA, U6 CC56-12SURKWA, U7 74HC165, U8 74HC165, U9 74HC595, Y1 Crystal

Commit message: layout changes
Parts:
- added H5: MountingHole_Pad, MountingHole:MountingHole_3.2mm_M3_DIN965_Pad, F.Cu at (70.9, 120.4)
- added H6: MountingHole_Pad, MountingHole:MountingHole_3.2mm_M3_DIN965_Pad, F.Cu at (147.2, 89.8)
- added J14: Conn_01x04_Male, Connector_PinHeader_2.54mm:PinHeader_1x04_P2.54mm_Vertical, F.Cu at (123.4, 185.8)
- moved J12 15.2 mm to (121.5, 87.8), turned to 90 degrees
- moved J8 6.54 mm to (69.6, 62.5)
- moved C3 2.50 mm to (147.2, 103.4)
- moved C4 2.50 mm to (147.2, 98.5)
Connections:
- J12 pad 3: /PC2 -> /PC3
- J12 pad 4: /PC0 -> /PC2
- J12 pad 6: /PC3 -> /PC0
Routing:
- net /PC1: track 35.8 -> 203.9 mm, vias 0 -> 2
- net /PC0: track 34.0 -> 202.0 mm, vias 0 -> 2
- net /PC2: track 53.4 -> 207.6 mm, vias 0 -> 2
- net /Buttons_Row_1_and_2/Serial_2: track 29.3 -> 165.3 mm, vias 0 -> 2
- net Net-(R32-Pad2): track 31.2 -> 131.0 mm
- net Net-(R33-Pad2): track 32.5 -> 113.2 mm, vias 0 -> 1
- net Net-(R34-Pad2): track 41.1 -> 95.4 mm, vias 0 -> 1
- net GND: track 92.0 -> 45.0 mm
- net +5V: track 117.5 -> 161.9 mm
- net /PD4: track 159.9 -> 194.0 mm, vias 0 -> 1
- net Net-(R30-Pad2): track 45.7 -> 77.0 mm, vias 1 -> 0
- net Net-(R29-Pad2): track 38.6 -> 64.3 mm, vias 1 -> 0
- net Net-(R35-Pad2): track 52.1 -> 77.1 mm, vias 0 -> 1
- net Net-(R31-Pad2): track 65.9 -> 89.7 mm
- net Net-(D9-Pad2): track 26.3 -> 45.7 mm, vias 1 -> 0
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
Commit message: moved crystal
Parts:
- added D13: Controll LED 1, LED_THT:LED_D5.0mm, F.Cu at (68.4, 125.3)
- added D14: Controll LED 2, LED_THT:LED_D5.0mm, F.Cu at (76.0, 125.3)
- added Q9: Q_PMOS_GDS, Package_TO_SOT_THT:TO-220-3_Horizontal_TabDown, F.Cu at (46.7, 54.7)
- added R64: 90R, Resistor_THT:R_Axial_DIN0207_L6.3mm_D2.5mm_P7.62mm_Horizontal, F.Cu at (89.1, 131.4)
- added R65: 90R, Resistor_THT:R_Axial_DIN0207_L6.3mm_D2.5mm_P7.62mm_Horizontal, F.Cu at (85.1, 123.8)
- J13: value Conn_01x06_Male -> Phase_Bitshifter
- J14: value Conn_01x04_Male -> Phase_Button_Decoder
- moved H5 36.6 mm to (35.4, 129.2)
- moved J3 29.0 mm to (71.1, 58.2)
- moved H6 18.8 mm to (151.8, 108.0)
- moved C3 11.4 mm to (136.8, 108.0)
- moved C4 11.4 mm to (136.8, 103.1)
- moved Y1 11.0 mm to (141.8, 103.1)
- moved Q6 7.44 mm to (126.7, 128.1)
- moved C10 7.34 mm to (60.5, 131.4)
- moved C11 7.34 mm to (94.5, 92.7)
- moved C12 7.34 mm to (94.5, 90.1)
- moved C13 7.34 mm to (58.0, 160.7)
- moved C15 7.34 mm to (58.0, 175.4)
- moved C16 7.34 mm to (58.0, 178.4)
- moved C17 7.34 mm to (58.0, 188.1)
- moved C18 7.34 mm to (58.0, 190.7)
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Connections:
- J10 pad 1: +5V -> Net-(J10-Pad1)
- J11 pad 1: +5V -> Net-(J10-Pad1)
- R2 pad 2: /RX -> /TX
- R3 pad 2: /TX -> /RX
- U1 pad 14: Net-(R2-Pad1) -> Net-(R3-Pad1)
- U1 pad 15: Net-(R3-Pad1) -> Net-(R2-Pad1)
- U1 pad 4: unconnected-(U1-Pad4) -> /PB3
- U1 pad 5: unconnected-(U1-Pad5) -> /PB4
- U11 pad 10: unconnected-(U11-Pad10) -> GND
- U11 pad 7: GND -> unconnected-(U11-Pad7)
- U7 pad 7: GND -> unconnected-(U7-Pad7)
- U8 pad 10: unconnected-(U8-Pad10) -> GND
- U8 pad 7: GND -> unconnected-(U8-Pad7)
Routing:
- net +5V: track 161.9 -> 233.5 mm, vias 1 -> 2
- net Net-(J10-Pad1): track 0.00 -> 26.9 mm
- net /PB3: track 0.00 -> 24.0 mm
- net Net-(D13-Pad1): track 0.00 -> 23.3 mm
- net GND: track 45.0 -> 65.1 mm
- net /PB4: track 0.00 -> 19.0 mm
- net /PB0: track 113.0 -> 131.4 mm
- net /MISO: track 47.6 -> 60.8 mm
- net /SCK: track 47.6 -> 58.3 mm
- net Net-(D14-Pad1): track 0.00 -> 9.72 mm
- net Net-(R2-Pad1): track 44.9 -> 54.5 mm
- net Net-(C3-Pad1): track 39.9 -> 31.1 mm
- net Net-(C4-Pad1): track 44.5 -> 35.7 mm
- net Net-(R3-Pad1): track 49.5 -> 56.3 mm
- net /PB2: track 152.6 -> 158.7 mm
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
Commit message: production gerber and new pictures
Parts:
- moved R59 12.4 mm to (93.9, 200.0), turned to -90 degrees
- moved R63 12.4 mm to (146.3, 200.0), turned to -90 degrees
- moved R56 12.4 mm to (54.6, 200.0), turned to -90 degrees
- moved R57 12.4 mm to (67.7, 200.0), turned to -90 degrees
- moved R58 12.4 mm to (80.8, 200.0), turned to -90 degrees
- moved R60 12.4 mm to (107.0, 200.0), turned to -90 degrees
- moved R61 12.4 mm to (120.1, 200.0), turned to -90 degrees
- moved R62 12.4 mm to (133.2, 200.0), turned to -90 degrees
Routing:
- net Net-(R57-Pad2): track 66.8 -> 64.4 mm
- net Net-(R62-Pad2): track 57.1 -> 54.6 mm
- net Net-(R61-Pad2): track 46.4 -> 43.9 mm
- net Net-(R60-Pad2): track 35.0 -> 32.5 mm
- net Net-(R58-Pad2): track 51.0 -> 48.5 mm
- net Net-(R63-Pad2): track 66.6 -> 64.1 mm
- net Net-(R59-Pad2): track 53.2 -> 50.7 mm
- net Net-(R56-Pad2): track 82.9 -> 80.4 mm
